Commit message: attached d435 & array error fix

File: ws_capstone/src/cma_urdf_description/urdf/cma_urdf.xacro (robot description, xacro)
@@ -1,493 +1,498 @@
 <?xml version="1.0" ?>
-<robot name="cma_urdf" xmlns:xacro="http://www.ros.org/wiki/xacro">
-<xacro:include filename="$(find cma_urdf_description)/urdf/materials.xacro" />
-<xacro:include filename="$(find cma_urdf_description)/urdf/cma_urdf.trans" />
-<xacro:include filename="$(find cma_urdf_description)/urdf/cma_urdf.gazebo" />
-<link name="base_link">
-  <inertial>
-    <origin rpy="0 0 0" xyz="9.621533355862818e-14 3.3453199900713086e-14 0.008001282197718517"/>
-    <mass value="106.9483036748442"/>
-    <inertia ixx="5.167281" ixy="0.0" ixz="-0.0" iyy="13.220959" iyz="-0.0" izz="18.383707"/>
-  </inertial>
-  <visual>
-    <origin rpy="0 0 0" xyz="0 0 0"/>
-    <geometry>
-      <mesh filename="package://cma_urdf_description/meshes/base_link.stl" scale="0.001 0.001 0.001"/>
-    </geometry>
-    <material name="silver"/>
-  </visual>
-  <collision>
-    <origin rpy="0 0 0" xyz="0 0 0"/>
-    <geometry>
-      <mesh filename="package://cma_urdf_description/meshes/base_link.stl" scale="0.001 0.001 0.001"/>
-    </geometry>
-  </collision>
-</link>
-<link name="robot_to_table_adp_1">
-  <inertial>
-    <origin rpy="0 0 0" xyz="-0.10160000000000019 -0.10160000000000002 0.01056181707210805"/>
-    <mass value="8.798853472720092"/>
-    <inertia ixx="0.03741" ixy="0.0" ixz="0.0" iyy="0.03741" iyz="-0.0" izz="0.07371"/>
-  </inertial>
-  <visual>
-    <origin rpy="0 0 0" xyz="-0.5842 -0.3556 -0.016"/>
-    <geometry>
-      <mesh filename="package://cma_urdf_description/meshes/robot_to_table_adp_1.stl" scale="0.001 0.001 0.001"/>
-    </geometry>
-    <material name="silver"/>
-  </visual>
-  <collision>
-    <origin rpy="0 0 0" xyz="-0.5842 -0.3556 -0.016"/>
-    <geometry>
-      <mesh filename="package://cma_urdf_description/meshes/robot_to_table_adp_1.stl" scale="0.001 0.001 0.001"/>
-    </geometry>
-  </collision>
-</link>
-<link name="Base_UR5_1">
-  <inertial>
-    <origin rpy="0 0 0" xyz="1.4232860621410381e-05 0.038282955879581804 0.05630526686916636"/>
-    <mass value="6.017293428658217"/>
-    <inertia ixx="0.090513" ixy="2e-06" ixz="4e-06" iyy="0.011877" iyz="0.01078" izz="0.09152"/>
-  </inertial>
-  <visual>
-    <origin rpy="0 0 0" xyz="-0.4826 -0.254 -0.046"/>
-    <geometry>
-      <mesh filename="package://cma_urdf_description/meshes/Base_UR5_1.stl" scale="0.001 0.001 0.001"/>
-    </geometry>
-    <material name="silver"/>
-  </visual>
-  <collision>
-    <origin rpy="0 0 0" xyz="-0.4826 -0.254 -0.046"/>
-    <geometry>
-      <mesh filename="package://cma_urdf_description/meshes/Base_UR5_1.stl" scale="0.001 0.001 0.001"/>
-    </geometry>
-  </collision>
-</link>
-<link name="Link1_UR5_1">
-  <inertial>
-    <origin rpy="0 0 0" xyz="-6.849514455620209e-09 -0.010909793967197823 0.06351880218055075"/>
-    <mass value="12.621938032794217"/>
-    <inertia ixx="0.030809" ixy="0.0" ixz="-0.0" iyy="0.027066" iyz="0.000743" izz="0.02624"/>
-  </inertial>
-  <visual>
-    <origin rpy="0 0 0" xyz="-0.4826 -0.254 -0.1451"/>
-    <geometry>
-      <mesh filename="package://cma_urdf_description/meshes/Link1_UR5_1.stl" scale="0.001 0.001 0.001"/>
-    </geometry>
-    <material name="silver"/>
-  </visual>
-  <collision>
-    <origin rpy="0 0 0" xyz="-0.4826 -0.254 -0.1451"/>
-    <geometry>
-      <mesh filename="package://cma_urdf_description/meshes/Link1_UR5_1.stl" scale="0.001 0.001 0.001"/>
-    </geometry>
-  </collision>
-</link>
-<link name="Link2_UR5_1">
-  <inertial>
-    <origin rpy="0 0 0" xyz="4.605402337265474e-09 -0.06350976997942634 0.21250002923894115"/>
-    <mass value="27.334504083061912"/>
-    <inertia ixx="1.110326" ixy="0.0" ixz="0.0" iyy="1.10119" iyz="0.0" izz="0.05819"/>
-  </inertial>
-  <visual>
-    <origin rpy="0 0 0" xyz="-0.4826 -0.1796 -0.2085"/>
-    <geometry>
-      <mesh filename="package://cma_urdf_description/meshes/Link2_UR5_1.stl" scale="0.001 0.001 0.001"/>
-    </geometry>
-    <material name="silver"/>
-  </visual>
-  <collision>
-    <origin rpy="0 0 0" xyz="-0.4826 -0.1796 -0.2085"/>
-    <geometry>
-      <mesh filename="package://cma_urdf_description/meshes/Link2_UR5_1.stl" scale="0.001 0.001 0.001"/>
-    </geometry>
-  </collision>
-</link>
-<link name="Link3_UR5_1">
-  <inertial>
-    <origin rpy="0 0 0" xyz="-2.9563169799406985e-06 0.057186964790381045 0.14791854418095085"/>
-    <mass value="14.0014424889426"/>
-    <inertia ixx="0.421335" ixy="1e-06" ixz="1.1e-05" iyy="0.417307" iyz="-0.027579" izz="0.02107"/>
-  </inertial>
-  <visual>
-    <origin rpy="0 0 0" xyz="-0.4826 -0.1796 -0.6335"/>
-    <geometry>
-      <mesh filename="package://cma_urdf_description/meshes/Link3_UR5_1.stl" scale="0.001 0.001 0.001"/>
-    </geometry>
-    <material name="silver"/>
-  </visual>
-  <collision>
-    <origin rpy="0 0 0" xyz="-0.4826 -0.1796 -0.6335"/>
-    <geometry>
-      <mesh filename="package://cma_urdf_description/meshes/Link3_UR5_1.stl" scale="0.001 0.001 0.001"/>
-    </geometry>
-  </collision>
-</link>
-<link name="Link4_UR5_1">
-  <inertial>
-    <origin rpy="0 0 0" xyz="7.862227992705417e-06 -0.062093450006130035 -0.002547992766358753"/>
-    <mass value="5.167091211713838"/>
-    <inertia ixx="0.008583" ixy="2e-06" ixz="1e-06" iyy="0.005396" iyz="-0.0002" izz="0.006947"/>
-  </inertial>
-  <visual>
-    <origin rpy="0 0 0" xyz="-0.4826 -0.2011 -1.02575"/>
-    <geometry>
-      <mesh filename="package://cma_urdf_description/meshes/Link4_UR5_1.stl" scale="0.001 0.001 0.001"/>
-    </geometry>
-    <material name="silver"/>
-  </visual>
-  <collision>
-    <origin rpy="0 0 0" xyz="-0.4826 -0.2011 -1.02575"/>
-    <geometry>
-      <mesh filename="package://cma_urdf_description/meshes/Link4_UR5_1.stl" scale="0.001 0.001 0.001"/>
-    </geometry>
-  </collision>
-</link>
-<link name="Link5_UR5_1">
-  <inertial>
-    <origin rpy="0 0 0" xyz="-9.684678712595929e-06 0.0031103043138043934 0.04584822329807814"/>
-    <mass value="4.229065191905357"/>
-    <inertia ixx="0.005491" ixy="1e-06" ixz="2e-06" iyy="0.003861" iyz="-5.8e-05" izz="0.00473"/>
-  </inertial>
-  <visual>
-    <origin rpy="0 0 0" xyz="-0.4826 -0.1207 -1.07205"/>
-    <geometry>
-      <mesh filename="package://cma_urdf_description/meshes/Link5_UR5_1.stl" scale="0.001 0.001 0.001"/>
-    </geometry>
-    <material name="silver"/>
-  </visual>
-  <collision>
-    <origin rpy="0 0 0" xyz="-0.4826 -0.1207 -1.07205"/>
-    <geometry>
-      <mesh filename="package://cma_urdf_description/meshes/Link5_UR5_1.stl" scale="0.001 0.001 0.001"/>
-    </geometry>
-  </collision>
-</link>
-<link name="Link6_UR5_1">
-  <inertial>
-    <origin rpy="0 0 0" xyz="4.89386309254769e-12 -0.0250238691012189 -1.7988520705225497e-05"/>
-    <mass value="1.7186317710700016"/>
-    <inertia ixx="0.000958" ixy="0.0" ixz="-0.0" iyy="0.001192" iyz="1e-06" izz="0.000964"/>
-  </inertial>
-  <visual>
-    <origin rpy="0 0 0" xyz="-0.4826 -0.0744 -1.12545"/>
-    <geometry>
-      <mesh filename="package://cma_urdf_description/meshes/Link6_UR5_1.stl" scale="0.001 0.001 0.001"/>
-    </geometry>
-    <material name="silver"/>
-  </visual>
-  <collision>
-    <origin rpy="0 0 0" xyz="-0.4826 -0.0744 -1.12545"/>
-    <geometry>
-      <mesh filename="package://cma_urdf_description/meshes/Link6_UR5_1.stl" scale="0.001 0.001 0.001"/>
-    </geometry>
-  </collision>
-</link>
-<link name="Defeatured_2F-85_PAD_OPEN_finger4m_1">
-  <inertial>
-    <origin rpy="0 0 0" xyz="0.014583483806780984 -0.01646459714685118 -0.009099999695404204"/>
-    <mass value="0.11326339019031978"/>
-    <inertia ixx="2.8e-05" ixy="9e-06" ixz="0.0" iyy="1.1e-05" iyz="0.0" izz="3.2e-05"/>
-  </inertial>
-  <visual>
-    <origin rpy="0 0 0" xyz="-0.414841 0.090726 -1.1345"/>
-    <geometry>
-      <mesh filename="package://cma_urdf_description/meshes/Defeatured_2F-85_PAD_OPEN_finger4m_1.stl" scale="0.001 0.001 0.001"/>
-    </geometry>
-    <material name="silver"/>
-  </visual>
-  <collision>
-    <origin rpy="0 0 0" xyz="-0.414841 0.090726 -1.1345"/>
-    <geometry>
-      <mesh filename="package://cma_urdf_description/meshes/Defeatured_2F-85_PAD_OPEN_finger4m_1.stl" scale="0.001 0.001 0.001"/>
-    </geometry>
-  </collision>
-</link>
-<link name="Defeatured_2F-85_PAD_OPEN_Finger1m_1">
-  <inertial>
-    <origin rpy="0 0 0" xyz="-0.029386708258091532 -0.011108198902811152 -0.0046933996965830005"/>
-    <mass value="0.1509168112436001"/>
-    <inertia ixx="4.5e-05" ixy="-1.5e-05" ixz="-0.0" iyy="3.4e-05" iyz="-0.0" izz="5.9e-05"/>
-  </inertial>
-  <visual>
-    <origin rpy="0 0 0" xyz="-0.451999 0.047305 -1.13015"/>
-    <geometry>
-      <mesh filename="package://cma_urdf_description/meshes/Defeatured_2F-85_PAD_OPEN_Finger1m_1.stl" scale="0.001 0.001 0.001"/>
-    </geometry>
-    <material name="silver"/>
-  </visual>
-  <collision>
-    <origin rpy="0 0 0" xyz="-0.451999 0.047305 -1.13015"/>
-    <geometry>
-      <mesh filename="package://cma_urdf_description/meshes/Defeatured_2F-85_PAD_OPEN_Finger1m_1.stl" scale="0.001 0.001 0.001"/>
-    </geometry>
-  </collision>
-</link>
-<link name="Defeatured_2F-85_PAD_OPEN_Finger1_1">
-  <inertial>
-    <origin rpy="0 0 0" xyz="0.029385642646017285 -0.011115663221872393 -0.004687336323244029"/>
-    <mass value="0.1508407345691058"/>
-    <inertia ixx="4.5e-05" ixy="1.5e-05" ixz="0.0" iyy="3.4e-05" iyz="-0.0" izz="5.9e-05"/>
-  </inertial>
-  <visual>
-    <origin rpy="0 0 0" xyz="-0.513201 0.047305 -1.13015"/>
-    <geometry>
-      <mesh filename="package://cma_urdf_description/meshes/Defeatured_2F-85_PAD_OPEN_Finger1_1.stl" scale="0.001 0.001 0.001"/>
-    </geometry>
-    <material name="silver"/>
-  </visual>
-  <collision>
-    <origin rpy="0 0 0" xyz="-0.513201 0.047305 -1.13015"/>
-    <geometry>
-      <mesh filename="package://cma_urdf_description/meshes/Defeatured_2F-85_PAD_OPEN_Finger1_1.stl" scale="0.001 0.001 0.001"/>
-    </geometry>
-  </collision>
-</link>
-<link name="Defeatured_2F-85_PAD_OPEN_finger4_1">
-  <inertial>
-    <origin rpy="0 0 0" xyz="-0.01458343021231212 -0.01646455128417476 -0.009100000304597122"/>
-    <mass value="0.11326339019032722"/>
-    <inertia ixx="2.8e-05" ixy="-9e-06" ixz="0.0" iyy="1.1e-05" iyz="-0.0" izz="3.2e-05"/>
-  </inertial>
-  <visual>
-    <origin rpy="0 0 0" xyz="-0.550359 0.090726 -1.1345"/>
-    <geometry>
-      <mesh filename="package://cma_urdf_description/meshes/Defeatured_2F-85_PAD_OPEN_finger4_1.stl" scale="0.001 0.001 0.001"/>
-    </geometry>
-    <material name="silver"/>
-  </visual>
-  <collision>
-    <origin rpy="0 0 0" xyz="-0.550359 0.090726 -1.1345"/>
-    <geometry>
-      <mesh filename="package://cma_urdf_description/meshes/Defeatured_2F-85_PAD_OPEN_finger4_1.stl" scale="0.001 0.001 0.001"/>
-    </geometry>
-  </collision>
-</link>
-<link name="Defeatured_2F-85_PAD_OPEN_base_1">
-  <inertial>
-    <origin rpy="0 0 0" xyz="0.02700117071233238 -0.032289625793831815 -0.015976537109387845"/>
-    <mass value="1.7710616874239076"/>
-    <inertia ixx="0.001378" ixy="-0.0" ixz="0.0" iyy="0.001054" iyz="1e-06" izz="0.00157"/>
-  </inertial>
-  <visual>
-    <origin rpy="0 0 0" xyz="-0.4556 -0.0076 -1.14145"/>
-    <geometry>
-      <mesh filename="package://cma_urdf_description/meshes/Defeatured_2F-85_PAD_OPEN_base_1.stl" scale="0.001 0.001 0.001"/>
-    </geometry>
-    <material name="silver"/>
-  </visual>
-  <collision>
-    <origin rpy="0 0 0" xyz="-0.4556 -0.0076 -1.14145"/>
-    <geometry>
-      <mesh filename="package://cma_urdf_description/meshes/Defeatured_2F-85_PAD_OPEN_base_1.stl" scale="0.001 0.001 0.001"/>
-    </geometry>
-  </collision>
-</link>
-<link name="urdf_Intel_RealSense_Depth_Camera_D435_v2_1">
-  <inertial>
-    <origin rpy="0 0 0" xyz="0.02101336009113891 -0.010035295733690969 6.117083960499592e-05"/>
-    <mass value="0.17091204023764017"/>
-    <inertia ixx="2e-05" ixy="1e-06" ixz="-0.0" iyy="0.000115" iyz="0.0" izz="0.000115"/>
-  </inertial>
-  <visual>
-    <origin rpy="0 0 0" xyz="-0.4601 -0.04665 -1.18745"/>
-    <geometry>
-      <mesh filename="package://cma_urdf_description/meshes/urdf_Intel_RealSense_Depth_Camera_D435_v2_1.stl" scale="0.001 0.001 0.001"/>
-    </geometry>
-    <material name="silver"/>
-  </visual>
-  <collision>
-    <origin rpy="0 0 0" xyz="-0.4601 -0.04665 -1.18745"/>
-    <geometry>
-      <mesh filename="package://cma_urdf_description/meshes/urdf_Intel_RealSense_Depth_Camera_D435_v2_1.stl" scale="0.001 0.001 0.001"/>
-    </geometry>
-  </collision>
-</link>
-<link name="camera_mount_1">
-  <inertial>
-    <origin rpy="0 0 0" xyz="5.835308347634793e-10 0.005987651723056972 0.03546806600852759"/>
-    <mass value="0.47184000408712967"/>
-    <inertia ixx="0.000606" ixy="0.0" ixz="-0.0" iyy="0.000964" iyz="0.0" izz="0.000369"/>
-  </inertial>
-  <visual>
-    <origin rpy="0 0 0" xyz="-0.4826 -0.04665 -1.12545"/>
-    <geometry>
-      <mesh filename="package://cma_urdf_description/meshes/camera_mount_1.stl" scale="0.001 0.001 0.001"/>
-    </geometry>
-    <material name="silver"/>
-  </visual>
-  <collision>
-    <origin rpy="0 0 0" xyz="-0.4826 -0.04665 -1.12545"/>
-    <geometry>
-      <mesh filename="package://cma_urdf_description/meshes/camera_mount_1.stl" scale="0.001 0.001 0.001"/>
-    </geometry>
-  </collision>
-</link>
-<link name="WRIST_CAMERA_20171116_v2_1">
-  <inertial>
-    <origin rpy="0 0 0" xyz="0.017204159491027715 -0.005175220524266128 -0.02290143817742174"/>
-    <mass value="0.547658826768176"/>
-    <inertia ixx="0.000308" ixy="-0.0" ixz="1e-06" iyy="0.000499" iyz="1e-05" izz="0.000221"/>
-  </inertial>
-  <visual>
-    <origin rpy="0 0 0" xyz="-0.464922 -0.0211 -1.143128"/>
-    <geometry>
-      <mesh filename="package://cma_urdf_description/meshes/WRIST_CAMERA_20171116_v2_1.stl" scale="0.001 0.001 0.001"/>
-    </geometry>
-    <material name="silver"/>
-  </visual>
-  <collision>
-    <origin rpy="0 0 0" xyz="-0.464922 -0.0211 -1.143128"/>
-    <geometry>
-      <mesh filename="package://cma_urdf_description/meshes/WRIST_CAMERA_20171116_v2_1.stl" scale="0.001 0.001 0.001"/>
-    </geometry>
-  </collision>
-</link>
-<link name="Defeatured_2F-85_PAD_OPEN_finger3m_1">
-  <inertial>
-    <origin rpy="0 0 0" xyz="0.0178887760737792 0.02120021807228656 -0.009100000000000552"/>
-    <mass value="0.07939275206386531"/>
-    <inertia ixx="2.5e-05" ixy="-1.1e-05" ixz="0.0" iyy="2.2e-05" iyz="-0.0" izz="2.3e-05"/>
-  </inertial>
-  <visual>
-    <origin rpy="0 0 0" xyz="-0.432743 0.097242 -1.1345"/>
-    <geometry>
-      <mesh filename="package://cma_urdf_description/meshes/Defeatured_2F-85_PAD_OPEN_finger3m_1.stl" scale="0.001 0.001 0.001"/>
-    </geometry>
-    <material name="silver"/>
-  </visual>
-  <collision>
-    <origin rpy="0 0 0" xyz="-0.432743 0.097242 -1.1345"/>
-    <geometry>
-      <mesh filename="package://cma_urdf_description/meshes/Defeatured_2F-85_PAD_OPEN_finger3m_1.stl" scale="0.001 0.001 0.001"/>
-    </geometry>
-  </collision>
-</link>
-<link name="Defeatured_2F-85_PAD_OPEN_finger3_1">
-  <inertial>
-    <origin rpy="0 0 0" xyz="-0.01818100035908876 0.020951006921311924 -0.009100000000000552"/>
-    <mass value="0.07939275206386531"/>
-    <inertia ixx="2.6e-05" ixy="1.1e-05" ixz="0.0" iyy="2.2e-05" iyz="0.0" izz="2.3e-05"/>
-  </inertial>
-  <visual>
-    <origin rpy="0 0 0" xyz="-0.532458 0.097242 -1.1345"/>
-    <geometry>
-      <mesh filename="package://cma_urdf_description/meshes/Defeatured_2F-85_PAD_OPEN_finger3_1.stl" scale="0.001 0.001 0.001"/>
-    </geometry>
-    <material name="silver"/>
-  </visual>
-  <collision>
-    <origin rpy="0 0 0" xyz="-0.532458 0.097242 -1.1345"/>
-    <geometry>
-      <mesh filename="package://cma_urdf_description/meshes/Defeatured_2F-85_PAD_OPEN_finger3_1.stl" scale="0.001 0.001 0.001"/>
-    </geometry>
-  </collision>
-</link>
-<joint name="Rigid10" type="fixed">
-  <origin rpy="0 0 0" xyz="0.5842 0.3556 0.016"/>
-  <parent link="base_link"/>
-  <child link="robot_to_table_adp_1"/>
-</joint>
-<joint name="Rigid11" type="fixed">
-  <origin rpy="0 0 0" xyz="-0.1016 -0.1016 0.03"/>
-  <parent link="robot_to_table_adp_1"/>
-  <child link="Base_UR5_1"/>
-</joint>
-<joint name="rev_a1" type="continuous">
-  <origin rpy="0 0 0" xyz="0.0 0.0 0.0991"/>
-  <parent link="Base_UR5_1"/>
-  <child link="Link1_UR5_1"/>
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
Commit message: camera position
camera position and colour for the arm

File: ws_capstone/src/cma_urdf_description/urdf/cma_urdf.xacro (robot description, xacro)
@@ -297,5 +297,5 @@
         <mesh filename="package://cma_urdf_description/meshes/urdf_Intel_RealSense_Depth_Camera_D435_v2_1.stl" scale="0.001 0.001 0.001"/>
       </geometry>
-      <material name="silver"/>
+      <material name="aluminum"/>
     </visual>
     <collision>
@@ -494,5 +494,5 @@
   </joint>
   <xacro:sensor_d435 name="realsense_d435" topics_ns="realsense_d435" parent="Link6_UR5_1" publish_pointcloud="true">
-    <origin xyz="0 0 0" rpy="0 0 0" />
+    <origin xyz="0 -0.04 0.05" rpy="0 0 -1.6" />
   </xacro:sensor_d435>
 </robot>

File: ws_capstone/src/cma_urdf_description/urdf/materials.xacro (robot description, xacro)
@@ -1,6 +1,9 @@
 <?xml version="1.0" ?>
 <robot name="cma_urdf" xmlns:xacro="http://www.ros.org/wiki/xacro" >
-<material name="silver">
-  <color rgba="0.700 0.700 0.700 1.000"/>
-</material>
+  <material name="silver">
+    <color rgba="0.700 0.700 0.700 1.000"/>
+  </material>
+  <material name="capstone_aluminum">
+    <color rgba="0.5 0.5 0.5 1"/>
+  </material>
 </robot>

Commit message: camera angle fixed

File: ws_capstone/src/cma_urdf_description/urdf/cma_urdf.xacro (robot description, xacro)
@@ -494,5 +494,5 @@
   </joint>
   <xacro:sensor_d435 name="realsense_d435" topics_ns="realsense_d435" parent="Link6_UR5_1" publish_pointcloud="true">
-    <origin xyz="0 -0.04 0.05" rpy="0 0 -1.6" />
+    <origin xyz="0 -0.04 0.05" rpy="0 0 -1.57079632679" />
   </xacro:sensor_d435>
 </robot>

Commit message: exact camera positioning

File: ws_capstone/src/cma_urdf_description/urdf/cma_urdf.xacro (robot description, xacro)
@@ -494,5 +494,5 @@
   </joint>
   <xacro:sensor_d435 name="realsense_d435" topics_ns="realsense_d435" parent="Link6_UR5_1" publish_pointcloud="true">
-    <origin xyz="0 -0.04 0.05" rpy="0 0 -1.57079632679" />
+    <origin xyz="0 -0.0379 0.0495" rpy="0 0 -1.57079632679" />
   </xacro:sensor_d435>
 </robot>

Commit message: removed old camera model

File: ws_capstone/src/cma_urdf_description/urdf/cma_urdf.xacro (robot description, xacro)
@@ -287,5 +287,5 @@
   </link>
   <link name="urdf_Intel_RealSense_Depth_Camera_D435_v2_1">
-    <inertial>
+    <!-- <inertial>
       <origin rpy="0 0 0" xyz="0.02101336009113891 -0.010035295733690969 6.117083960499592e-05"/>
       <mass value="0.17091204023764017"/>
@@ -304,5 +304,5 @@
         <mesh filename="package://cma_urdf_description/meshes/urdf_Intel_RealSense_Depth_Camera_D435_v2_1.stl" scale="0.001 0.001 0.001"/>
       </geometry>
-    </collision>
+    </collision> -->
   </link>
   <link name="camera_mount_1">
@@ -494,4 +494,5 @@
   </joint>
   <xacro:sensor_d435 name="realsense_d435" topics_ns="realsense_d435" parent="Link6_UR5_1" publish_pointcloud="true">
+    <!-- <origin xyz="0 -0.02775 0.062" rpy="0 0 -1.57079632679" /> -->
     <origin xyz="0 -0.0379 0.0495" rpy="0 0 -1.57079632679" />
   </xacro:sensor_d435>

Commit message: removed inertial property from base_link
gets rid of error

File: ws_capstone/src/cma_urdf_description/urdf/cma_urdf.xacro (robot description, xacro)
@@ -7,9 +7,9 @@
   <xacro:include filename="$(find realsense2_description)/urdf/_d435.urdf.xacro"/>
   <link name="base_link">
-    <inertial>
+    <!-- <inertial>
       <origin rpy="0 0 0" xyz="9.621533355862818e-14 3.3453199900713086e-14 0.008001282197718517"/>
       <mass value="106.9483036748442"/>
       <inertia ixx="5.167281" ixy="0.0" ixz="-0.0" iyy="13.220959" iyz="-0.0" izz="18.383707"/>
-    </inertial>
+    </inertial> -->
     <visual>
       <origin rpy="0 0 0" xyz="0 0 0"/>

Commit message: fixed base to world

File: ws_capstone/src/cma_urdf_description/urdf/cma_urdf.xacro (robot description, xacro)
@@ -6,4 +6,5 @@
   <xacro:include filename="$(find cma_urdf_description)/urdf/cma_urdf.gazebo" />
   <xacro:include filename="$(find realsense2_description)/urdf/_d435.urdf.xacro"/>
+  <link name="world" />
   <link name="base_link">
     <!-- <inertial>
@@ -386,4 +387,8 @@
     </collision>
   </link>
+  <joint name="base_to_world_link" type="fixed">
+    <parent link="world"/>
+    <child link="base_link"/>
+  </joint>
   <joint name="Rigid10" type="fixed">
     <origin rpy="0 0 0" xyz="0.5842 0.3556 0.016"/>
