Commit message: attempt gripper fix

File: ws_capstone/src/robotiq_85_description/urdf/robotiq_85_gripper.transmission.xacro (robot description, xacro)
@@ -68,18 +68,18 @@
                 <joint>${prefix}robotiq_85_left_knuckle_joint</joint>
                 <mimicJoint>${prefix}robotiq_85_right_knuckle_joint</mimicJoint>
-                <multiplier>1.0</multiplier>
-                <offset>0.0</offset>
+                <!-- <multiplier>1.0</multiplier>
+                <offset>0.0</offset> -->
             </plugin>
             <plugin filename="libroboticsgroup_gazebo_mimic_joint_plugin.so" name="${prefix}mimic_robotiq_85_2">
                 <joint>${prefix}robotiq_85_left_knuckle_joint</joint>
                 <mimicJoint>${prefix}robotiq_85_left_inner_knuckle_joint</mimicJoint>
-                <multiplier>1.0</multiplier>
-                <offset>0.0</offset>
+                <!-- <multiplier>1.0</multiplier>
+                <offset>0.0</offset> -->
             </plugin>
             <plugin filename="libroboticsgroup_gazebo_mimic_joint_plugin.so" name="${prefix}mimic_robotiq_85_3">
                 <joint>${prefix}robotiq_85_left_knuckle_joint</joint>
                 <mimicJoint>${prefix}robotiq_85_right_inner_knuckle_joint</mimicJoint>
-                <multiplier>1.0</multiplier>
-                <offset>0.0</offset>
+                <!-- <multiplier>1.0</multiplier>
+                <offset>0.0</offset> -->
             </plugin>
             <plugin filename="libroboticsgroup_gazebo_mimic_joint_plugin.so" name="${prefix}mimic_robotiq_85_4">
@@ -87,5 +87,5 @@
                 <mimicJoint>${prefix}robotiq_85_left_finger_tip_joint</mimicJoint>
                 <multiplier>-1.0</multiplier>
-                <offset>0.0</offset>
+                <!-- <offset>0.0</offset> -->
             </plugin>
             <plugin filename="libroboticsgroup_gazebo_mimic_joint_plugin.so" name="${prefix}mimic_robotiq_85_5">
@@ -93,9 +93,8 @@
                 <mimicJoint>${prefix}robotiq_85_right_finger_tip_joint</mimicJoint>
                 <multiplier>-1.0</multiplier>
-                <offset>0.0</offset>
+                <!-- <offset>0.0</offset> -->
             </plugin>
         </gazebo>
         <gazebo reference="${prefix}robotiq_85_left_finger_link">
-            <!-- <material>Gazebo/FlatBlack</material> -->
             <mu1>0.2</mu1>
             <mu2>0.2</mu2>
@@ -103,5 +102,4 @@
         </gazebo>
         <gazebo reference="${prefix}robotiq_85_right_finger_link">
-            <!-- <material>Gazebo/FlatBlack</material> -->
             <mu1>0.2</mu1>
             <mu2>0.2</mu2>

File: ws_capstone/src/robotiq_85_description/urdf/robotiq_85_gripper.urdf.xacro (robot description, xacro)
@@ -94,5 +94,5 @@
             <child link="${prefix}robotiq_85_right_finger_link"/>
             <!-- added -->
-            <axis xyz="0 1 0"/>
+            <axis xyz="0 0 1"/>
             <!-- added -->
             <origin xyz="-0.00408552455 -0.03148604435 0.0" rpy="0 0 0" />

File: ws_capstone/src/robotiq_85_description/urdf/robotiq_85_gripper.xacro (robot description, xacro)
@@ -34,6 +34,6 @@
                      izx = "0.000000" izy = "0.000000" izz = "0.000001" />
         </inertial>
-    </link> -->
-    <!-- <xacro:robotiq_85_gripper prefix="" parent="gripper_root_link" >
+    </link>
+    <xacro:robotiq_85_gripper prefix="" parent="gripper_root_link" >
         <origin xyz="0.05 0 0.85" rpy="0 0 0"/>
     </xacro:robotiq_85_gripper> -->

Commit message: gripper working!

File: ws_capstone/src/robotiq_85_description/urdf/robotiq_85_gripper.transmission.xacro (robot description, xacro)
@@ -65,36 +65,76 @@
         <gazebo>
             <!-- loading plugin: mimic joints works in gazebo now -->
-            <plugin filename="libroboticsgroup_gazebo_mimic_joint_plugin.so" name="${prefix}mimic_robotiq_85_1">
+            <plugin filename="libroboticsgroup_upatras_gazebo_mimic_joint_plugin.so" name="${prefix}mimic_robotiq_85_1">
                 <joint>${prefix}robotiq_85_left_knuckle_joint</joint>
                 <mimicJoint>${prefix}robotiq_85_right_knuckle_joint</mimicJoint>
+                <maxEffort>1000</maxEffort>
                 <!-- <multiplier>1.0</multiplier>
                 <offset>0.0</offset> -->
             </plugin>
-            <plugin filename="libroboticsgroup_gazebo_mimic_joint_plugin.so" name="${prefix}mimic_robotiq_85_2">
+            <plugin filename="libroboticsgroup_upatras_gazebo_mimic_joint_plugin.so" name="${prefix}mimic_robotiq_85_2">
                 <joint>${prefix}robotiq_85_left_knuckle_joint</joint>
                 <mimicJoint>${prefix}robotiq_85_left_inner_knuckle_joint</mimicJoint>
+                <maxEffort>1000</maxEffort>
                 <!-- <multiplier>1.0</multiplier>
                 <offset>0.0</offset> -->
             </plugin>
-            <plugin filename="libroboticsgroup_gazebo_mimic_joint_plugin.so" name="${prefix}mimic_robotiq_85_3">
+            <plugin filename="libroboticsgroup_upatras_gazebo_mimic_joint_plugin.so" name="${prefix}mimic_robotiq_85_3">
                 <joint>${prefix}robotiq_85_left_knuckle_joint</joint>
                 <mimicJoint>${prefix}robotiq_85_right_inner_knuckle_joint</mimicJoint>
+                <maxEffort>1000</maxEffort>
                 <!-- <multiplier>1.0</multiplier>
                 <offset>0.0</offset> -->
             </plugin>
-            <plugin filename="libroboticsgroup_gazebo_mimic_joint_plugin.so" name="${prefix}mimic_robotiq_85_4">
+            <plugin filename="libroboticsgroup_upatras_gazebo_mimic_joint_plugin.so" name="${prefix}mimic_robotiq_85_4">
                 <joint>${prefix}robotiq_85_left_knuckle_joint</joint>
                 <mimicJoint>${prefix}robotiq_85_left_finger_tip_joint</mimicJoint>
+                <maxEffort>1000</maxEffort>
                 <multiplier>-1.0</multiplier>
                 <!-- <offset>0.0</offset> -->
             </plugin>
-            <plugin filename="libroboticsgroup_gazebo_mimic_joint_plugin.so" name="${prefix}mimic_robotiq_85_5">
+            <plugin filename="libroboticsgroup_upatras_gazebo_mimic_joint_plugin.so" name="${prefix}mimic_robotiq_85_5">
                 <joint>${prefix}robotiq_85_left_knuckle_joint</joint>
                 <mimicJoint>${prefix}robotiq_85_right_finger_tip_joint</mimicJoint>
+                <maxEffort>1000</maxEffort>
                 <multiplier>-1.0</multiplier>
                 <!-- <offset>0.0</offset> -->
             </plugin>
         </gazebo>
+        <!-- <gazebo reference="${prefix}robotiq_85_base_link">
+            <mu1>0.2</mu1>
+            <mu2>0.2</mu2>
+            <selfCollide>false</selfCollide>
+        </gazebo> -->
+        <gazebo reference="${prefix}robotiq_85_left_inner_knuckle_link">
+            <mu1>0.2</mu1>
+            <mu2>0.2</mu2>
+            <selfCollide>false</selfCollide>
+        </gazebo>
+        <gazebo reference="${prefix}robotiq_85_left_finger_tip_link">
+            <mu1>0.2</mu1>
+            <mu2>0.2</mu2>
+            <selfCollide>false</selfCollide>
+        </gazebo>
+        <gazebo reference="${prefix}robotiq_85_left_knuckle_link">
+            <mu1>0.2</mu1>
+            <mu2>0.2</mu2>
+            <selfCollide>false</selfCollide>
+        </gazebo>
         <gazebo reference="${prefix}robotiq_85_left_finger_link">
+            <mu1>0.2</mu1>
+            <mu2>0.2</mu2>
+            <selfCollide>false</selfCollide>
+        </gazebo>
+        <gazebo reference="${prefix}robotiq_85_right_inner_knuckle_link">
+            <mu1>0.2</mu1>
+            <mu2>0.2</mu2>
+            <selfCollide>false</selfCollide>
+        </gazebo>
+        <gazebo reference="${prefix}robotiq_85_right_finger_tip_link">
+            <mu1>0.2</mu1>
+            <mu2>0.2</mu2>
+            <selfCollide>false</selfCollide>
+        </gazebo>
+        <gazebo reference="${prefix}robotiq_85_right_knuckle_link">
             <mu1>0.2</mu1>
             <mu2>0.2</mu2>

File: ws_capstone/src/robotiq_85_description/urdf/robotiq_85_gripper.urdf.xacro (robot description, xacro)
@@ -86,5 +86,5 @@
             <child link="${prefix}robotiq_85_left_finger_link"/>
             <!-- added -->
-            <axis xyz="0 0 1"/>
+            <axis xyz="0 1 0"/>
             <!-- added -->
             <origin xyz="-0.00408552455 -0.03148604435 0.0" rpy="0 0 0" />
@@ -94,5 +94,5 @@
             <child link="${prefix}robotiq_85_right_finger_link"/>
             <!-- added -->
-            <axis xyz="0 0 1"/>
+            <axis xyz="0 1 0"/>
             <!-- added -->
             <origin xyz="-0.00408552455 -0.03148604435 0.0" rpy="0 0 0" />
@@ -110,4 +110,10 @@
             </collision>
             <inertial>
+                <!-- <mass value="0" />
+                <origin xyz="0.0 0.0 0.0" />
+                <inertia ixx = "0" ixy = "0" ixz = "0"
+                         iyx = "0" iyy = "0" iyz = "0"
+                         izx = "0" izy = "0" izz = "0" />
+            </inertial> -->
                 <mass value="0.027309" />
                 <origin xyz="0.0 0.0 0.0" />
@@ -129,5 +135,11 @@
             </collision>
             <inertial>
-                <mass value="0.027309" />
+                <!-- <mass value="0" />
+                <origin xyz="0.0 0.0 0.0" />
+                <inertia ixx = "0" ixy = "0" ixz = "0"
+                         iyx = "0" iyy = "0" iyz = "0"
+                         izx = "0" izy = "0" izz = "0" />
+            </inertial> -->
+            <mass value="0.027309" />
                 <origin xyz="0.0 0.0 0.0" />
                 <inertia ixx = "0.000003" ixy = "-0.000002" ixz = "0.000000"

Commit message: changes to gripper and capstone_scheduler

File: ws_capstone/src/robotiq_85_description/urdf/robotiq_85_gripper.transmission.xacro (robot description, xacro)
@@ -114,5 +114,5 @@
             <mu1>0.2</mu1>
             <mu2>0.2</mu2>
-            <selfCollide>false</selfCollide>
+            <selfCollide>true</selfCollide>
         </gazebo>
         <gazebo reference="${prefix}robotiq_85_left_knuckle_link">
@@ -134,5 +134,5 @@
             <mu1>0.2</mu1>
             <mu2>0.2</mu2>
-            <selfCollide>false</selfCollide>
+            <selfCollide>true</selfCollide>
         </gazebo>
         <gazebo reference="${prefix}robotiq_85_right_knuckle_link">

File: ws_capstone/src/robotiq_85_description/urdf/robotiq_85_gripper.urdf.xacro (robot description, xacro)
@@ -99,5 +99,5 @@
         </joint>
         <link name="${prefix}robotiq_85_left_finger_link">
-            <visual>
+            <!-- <visual>
                 <geometry>
                     <mesh filename="package://robotiq_85_description/meshes/visual/robotiq_85_finger_link.dae"/>
@@ -110,10 +110,4 @@
             </collision>
             <inertial>
-                <!-- <mass value="0" />
-                <origin xyz="0.0 0.0 0.0" />
-                <inertia ixx = "0" ixy = "0" ixz = "0"
-                         iyx = "0" iyy = "0" iyz = "0"
-                         izx = "0" izy = "0" izz = "0" />
-            </inertial> -->
                 <mass value="0.027309" />
                 <origin xyz="0.0 0.0 0.0" />
@@ -121,8 +115,8 @@
                          iyx = "-0.000002" iyy = "0.000021" iyz = "0.000000"
                          izx = "0.000000" izy = "0.000000" izz = "0.000020" />
-            </inertial>
+            </inertial> -->
         </link>
         <link name="${prefix}robotiq_85_right_finger_link">
-            <visual>
+            <!-- <visual>
                 <geometry>
                     <mesh filename="package://robotiq_85_description/meshes/visual/robotiq_85_finger_link.dae"/>
@@ -135,10 +129,4 @@
             </collision>
             <inertial>
-                <!-- <mass value="0" />
-                <origin xyz="0.0 0.0 0.0" />
-                <inertia ixx = "0" ixy = "0" ixz = "0"
-                         iyx = "0" iyy = "0" iyz = "0"
-                         izx = "0" izy = "0" izz = "0" />
-            </inertial> -->
             <mass value="0.027309" />
                 <origin xyz="0.0 0.0 0.0" />
@@ -146,5 +134,5 @@
                          iyx = "-0.000002" iyy = "0.000021" iyz = "0.000000"
                          izx = "0.000000" izy = "0.000000" izz = "0.000020" />
-            </inertial>
+            </inertial> -->
         </link>
         <joint name="${prefix}robotiq_85_left_inner_knuckle_joint" type="continuous">

Commit message: gripper cleanup

File: ws_capstone/src/robotiq_85_description/urdf/robotiq_85_gripper.transmission.xacro (robot description, xacro)
@@ -68,5 +68,5 @@
                 <joint>${prefix}robotiq_85_left_knuckle_joint</joint>
                 <mimicJoint>${prefix}robotiq_85_right_knuckle_joint</mimicJoint>
-                <maxEffort>1000</maxEffort>
+                <maxEffort>10</maxEffort>
                 <!-- <multiplier>1.0</multiplier>
                 <offset>0.0</offset> -->
@@ -75,5 +75,5 @@
                 <joint>${prefix}robotiq_85_left_knuckle_joint</joint>
                 <mimicJoint>${prefix}robotiq_85_left_inner_knuckle_joint</mimicJoint>
-                <maxEffort>1000</maxEffort>
+                <maxEffort>10</maxEffort>
                 <!-- <multiplier>1.0</multiplier>
                 <offset>0.0</offset> -->
@@ -82,5 +82,5 @@
                 <joint>${prefix}robotiq_85_left_knuckle_joint</joint>
                 <mimicJoint>${prefix}robotiq_85_right_inner_knuckle_joint</mimicJoint>
-                <maxEffort>1000</maxEffort>
+                <maxEffort>10</maxEffort>
                 <!-- <multiplier>1.0</multiplier>
                 <offset>0.0</offset> -->
@@ -89,5 +89,5 @@
                 <joint>${prefix}robotiq_85_left_knuckle_joint</joint>
                 <mimicJoint>${prefix}robotiq_85_left_finger_tip_joint</mimicJoint>
-                <maxEffort>1000</maxEffort>
+                <maxEffort>10</maxEffort>
                 <multiplier>-1.0</multiplier>
                 <!-- <offset>0.0</offset> -->
@@ -96,5 +96,5 @@
                 <joint>${prefix}robotiq_85_left_knuckle_joint</joint>
                 <mimicJoint>${prefix}robotiq_85_right_finger_tip_joint</mimicJoint>
-                <maxEffort>1000</maxEffort>
+                <maxEffort>10</maxEffort>
                 <multiplier>-1.0</multiplier>
                 <!-- <offset>0.0</offset> -->

File: ws_capstone/src/robotiq_85_description/urdf/robotiq_85_gripper.urdf.xacro (robot description, xacro)
@@ -34,5 +34,5 @@
             <axis xyz="0 0 1"/>
             <origin rpy="${pi} 0.0 0.0" xyz="0.05490451627 0.03060114443 0.0"/>
-            <limit lower="0.0" upper="0.8" velocity="2.0" effort="1000"/>
+            <limit lower="0.0" upper="0.8" velocity="2.0" effort="10"/>
         </joint>
         <joint name="${prefix}robotiq_85_right_knuckle_joint" type="continuous">
@@ -86,5 +86,5 @@
             <child link="${prefix}robotiq_85_left_finger_link"/>
             <!-- added -->
-            <axis xyz="0 1 0"/>
+            <!-- <axis xyz="0 1 0"/> -->
             <!-- added -->
             <origin xyz="-0.00408552455 -0.03148604435 0.0" rpy="0 0 0" />
@@ -94,5 +94,5 @@
             <child link="${prefix}robotiq_85_right_finger_link"/>
             <!-- added -->
-            <axis xyz="0 1 0"/>
+            <!-- <axis xyz="0 1 0"/> -->
             <!-- added -->
             <origin xyz="-0.00408552455 -0.03148604435 0.0" rpy="0 0 0" />
