Commit message: flat table, added joint limits, and gripper attach changes

File: ws_capstone/src/urdf_descriptions_plugins/cma_urdf_description/urdf/cma_urdf.xacro (robot description, xacro)
@@ -18,5 +18,5 @@
       <origin rpy="0 0 0" xyz="0 0 0"/>
       <geometry>
-        <mesh filename="package://cma_urdf_description/meshes/base_link.stl" scale="0.001 0.001 0.001"/>
+        <mesh filename="package://cma_urdf_description/meshes/table2.dae" scale="0.01 0.01 0.01"/>
       </geometry>
       <material name="silver"/>
@@ -25,5 +25,5 @@
       <origin rpy="0 0 0" xyz="0 0 0"/>
       <geometry>
-        <mesh filename="package://cma_urdf_description/meshes/base_link.stl" scale="0.001 0.001 0.001"/>
+        <mesh filename="package://cma_urdf_description/meshes/table.stl" scale="0.001 0.001 0.001"/>
       </geometry>
     </collision>
@@ -403,39 +403,45 @@
     <child link="Base_UR5_1"/>
   </joint>
-  <joint name="rev_a1" type="continuous">
+  <joint name="rev_a1" type="revolute">
     <origin rpy="0 0 0" xyz="0.0 0.0 0.0991"/>
     <parent link="Base_UR5_1"/>
     <child link="Link1_UR5_1"/>
     <axis xyz="-0.0 0.0 -1.0"/>
-  </joint>
-  <joint name="rev_a2" type="continuous">
+    <limit lower="-3.1415" upper="3.1415" velocity="5" effort="1000"/>
+  </joint>
+  <joint name="rev_a2" type="revolute">
     <origin rpy="0 0 0" xyz="0.0 -0.0744 0.0634"/>
     <parent link="Link1_UR5_1"/>
     <child link="Link2_UR5_1"/>
     <axis xyz="-0.0 1.0 0.0"/>
-  </joint>
-  <joint name="rev_a3" type="continuous">
+    <limit lower="0" upper="3.1415" velocity="5" effort="1000"/>
+  </joint>
+  <joint name="rev_a3" type="revolute">
     <origin rpy="0 0 0" xyz="0.0 0.0 0.425"/>
     <parent link="Link2_UR5_1"/>
     <child link="Link3_UR5_1"/>
     <axis xyz="0.0 1.0 -0.0"/>
-  </joint>
-  <joint name="rev_a4" type="continuous">
+    <limit lower="0.0" upper="3.1415" velocity="5" effort="1000"/>
+  </joint>
+  <joint name="rev_a4" type="revolute">
     <origin rpy="0 0 0" xyz="0.0 0.0215 0.39225"/>
     <parent link="Link3_UR5_1"/>
     <child link="Link4_UR5_1"/>
     <axis xyz="-0.0 -1.0 -0.0"/>
-  </joint>
-  <joint name="rev_a5" type="continuous">
+    <limit lower="-3.1415" upper="3.1415" velocity="5" effort="1000"/>
+  </joint>
+  <joint name="rev_a5" type="revolute">
     <origin rpy="0 0 0" xyz="0.0 -0.0804 0.0463"/>
     <parent link="Link4_UR5_1"/>
     <child link="Link5_UR5_1"/>
     <axis xyz="-0.0 -0.0 1.0"/>
-  </joint>
-  <joint name="rev_a6" type="continuous">
+    <limit lower="-3.1415" upper="3.1415" velocity="5" effort="1000"/>
+  </joint>
+  <joint name="rev_a6" type="revolute">
     <origin rpy="0 0 0" xyz="0.0 -0.0463 0.0534"/>
     <parent link="Link5_UR5_1"/>
     <child link="Link6_UR5_1"/>
     <axis xyz="0.0 -1.0 -0.0"/>
+    <limit lower="-3.1415" upper="3.1415" velocity="5" effort="1000"/>
   </joint>
   <!-- <joint name="rev_grp" type="revolute">

File: ws_capstone/src/urdf_descriptions_plugins/robotiq_85_description/urdf/robotiq_85_gripper.transmission.xacro (robot description, xacro)
@@ -68,5 +68,5 @@
                 <joint>${prefix}robotiq_85_left_knuckle_joint</joint>
                 <mimicJoint>${prefix}robotiq_85_right_knuckle_joint</mimicJoint>
-                <maxEffort>10</maxEffort>
+                <maxEffort>9.01</maxEffort>
                 <!-- <multiplier>1.0</multiplier>
                 <offset>0.0</offset> -->
@@ -75,5 +75,5 @@
                 <joint>${prefix}robotiq_85_left_knuckle_joint</joint>
                 <mimicJoint>${prefix}robotiq_85_left_inner_knuckle_joint</mimicJoint>
-                <maxEffort>10</maxEffort>
+                <maxEffort>9.01</maxEffort>
                 <!-- <multiplier>1.0</multiplier>
                 <offset>0.0</offset> -->
@@ -82,5 +82,5 @@
                 <joint>${prefix}robotiq_85_left_knuckle_joint</joint>
                 <mimicJoint>${prefix}robotiq_85_right_inner_knuckle_joint</mimicJoint>
-                <maxEffort>10</maxEffort>
+                <maxEffort>9.01</maxEffort>
                 <!-- <multiplier>1.0</multiplier>
                 <offset>0.0</offset> -->
@@ -89,5 +89,5 @@
                 <joint>${prefix}robotiq_85_left_knuckle_joint</joint>
                 <mimicJoint>${prefix}robotiq_85_left_finger_tip_joint</mimicJoint>
-                <maxEffort>10</maxEffort>
+                <maxEffort>9.01</maxEffort>
                 <multiplier>-1.0</multiplier>
                 <!-- <offset>0.0</offset> -->
@@ -96,5 +96,5 @@
                 <joint>${prefix}robotiq_85_left_knuckle_joint</joint>
                 <mimicJoint>${prefix}robotiq_85_right_finger_tip_joint</mimicJoint>
-                <maxEffort>10</maxEffort>
+                <maxEffort>9.01</maxEffort>
                 <multiplier>-1.0</multiplier>
                 <!-- <offset>0.0</offset> -->

File: ws_capstone/src/urdf_descriptions_plugins/robotiq_85_description/urdf/robotiq_85_gripper.urdf.xacro (robot description, xacro)
@@ -34,5 +34,5 @@
             <axis xyz="0 0 1"/>
             <origin rpy="${pi} 0.0 0.0" xyz="0.05490451627 0.03060114443 0.0"/>
-            <limit lower="0.0" upper="0.8" velocity="2.0" effort="10"/>
+            <limit lower="0.0" upper="0.8" velocity="2.0" effort="9.01"/>
             <dynamics friction="9"/>
         </joint>
@@ -42,7 +42,8 @@
             <axis xyz="0 0 1"/>
             <origin rpy="0.0 0.0 0.0" xyz="0.05490451627 -0.03060114443 0.0"/>
-            <limit lower="-3.14" upper="3.14" velocity="2" effort="1000"/>
+            <limit lower="-3.14" upper="3.14" velocity="2" effort="9.01"/>
             <mimic joint="${prefix}robotiq_85_left_knuckle_joint"/>
             <!-- <dynamics damping="0.7"/> -->
+            <dynamics friction="9"/>
         </joint>
         <link name="${prefix}robotiq_85_left_knuckle_link">
@@ -92,4 +93,5 @@
             <origin xyz="-0.00408552455 -0.03148604435 0.0" rpy="0 0 0" />
             <!-- <dynamics damping="0.7"/> -->
+            <dynamics friction="9"/>
         </joint>
         <joint name="${prefix}robotiq_85_right_finger_joint" type="continuous">
@@ -101,4 +103,5 @@
             <origin xyz="-0.00408552455 -0.03148604435 0.0" rpy="0 0 0" />
             <!-- <dynamics damping="0.7"/> -->
+            <dynamics friction="9"/>
         </joint>
         <link name="${prefix}robotiq_85_left_finger_link">
@@ -145,7 +148,8 @@
             <axis xyz="0 0 1"/>
             <origin xyz="0.06142 0.0127 0" rpy="${pi} 0.0 0.0" />
-            <limit lower="-3.14" upper="3.14" velocity="2" effort="10"/>
+            <limit lower="-3.14" upper="3.14" velocity="2" effort="9.01"/>
             <mimic joint="${prefix}robotiq_85_left_knuckle_joint" offset="0"/>
             <!-- <dynamics damping="0.7"/> -->
+            <dynamics friction="9"/>
         </joint>
         <joint name="${prefix}robotiq_85_right_inner_knuckle_joint" type="continuous">
@@ -154,7 +158,8 @@
             <axis xyz="0 0 1"/>
             <origin xyz="0.06142 -0.0127 0" rpy="0 0 0"/>
-            <limit lower="-3.14" upper="3.14" velocity="2" effort="10"/>
+            <limit lower="-3.14" upper="3.14" velocity="2" effort="9.01"/>
             <mimic joint="${prefix}robotiq_85_left_knuckle_joint" offset="0"/>
             <!-- <dynamics damping="0.7"/> -->
+            <dynamics friction="9"/>
         </joint>
         <link name="${prefix}robotiq_85_left_inner_knuckle_link">
@@ -201,7 +206,8 @@
             <axis xyz="0 0 1"/>
             <origin xyz="0.04303959807 -0.03759940821 0.0" rpy="0.0 0.0 0.0"/>
-            <limit lower="-3.14" upper="3.14" velocity="2" effort="10"/>
+            <limit lower="-3.14" upper="3.14" velocity="2" effort="9.01"/>
             <mimic joint="${prefix}robotiq_85_left_knuckle_joint" multiplier="-1"/>
             <!-- <dynamics damping="0.7"/> -->
+            <dynamics friction="9"/>
         </joint>
         <joint name="${prefix}robotiq_85_right_finger_tip_joint" type="continuous">
@@ -210,7 +216,8 @@
             <axis xyz="0 0 1"/>
             <origin rpy="0.0 0.0 0.0" xyz="0.04303959807 -0.03759940821  0.0"/>
-            <limit lower="-3.14" upper="3.14" velocity="2" effort="10"/>
+            <limit lower="-3.14" upper="3.14" velocity="2" effort="9.01"/>
             <mimic joint="${prefix}robotiq_85_left_knuckle_joint" multiplier="-1"/>
             <!-- <dynamics damping="0.7"/> -->
+            <dynamics friction="9"/>
         </joint>
         <link name="${prefix}robotiq_85_left_finger_tip_link">

Commit message: adjusted joint limits and added move sweep to look for object

File: ws_capstone/src/urdf_descriptions_plugins/cma_urdf_description/urdf/cma_urdf.xacro (robot description, xacro)
@@ -408,5 +408,5 @@
     <child link="Link1_UR5_1"/>
     <axis xyz="-0.0 0.0 -1.0"/>
-    <limit lower="-3.1415" upper="3.1415" velocity="5" effort="1000"/>
+    <limit lower="0" upper="6.28318530718" velocity="5" effort="1000"/>
   </joint>
   <joint name="rev_a2" type="revolute">
@@ -415,5 +415,5 @@
     <child link="Link2_UR5_1"/>
     <axis xyz="-0.0 1.0 0.0"/>
-    <limit lower="0" upper="3.1415" velocity="5" effort="1000"/>
+    <limit lower="-1.57079632679" upper="3.1415" velocity="5" effort="1000"/>
   </joint>
   <joint name="rev_a3" type="revolute">
@@ -436,5 +436,5 @@
     <child link="Link5_UR5_1"/>
     <axis xyz="-0.0 -0.0 1.0"/>
-    <limit lower="-3.1415" upper="3.1415" velocity="5" effort="1000"/>
+    <limit lower="0" upper="3.1415" velocity="5" effort="1000"/>
   </joint>
   <joint name="rev_a6" type="revolute">
