Commit message: gripper kind of gripping and general cleanup

File: ws_capstone/src/urdf_descriptions_plugins/robotiq_85_description/urdf/robotiq_85_gripper.transmission.xacro (robot description, xacro)
@@ -5,9 +5,9 @@
             <type>transmission_interface/SimpleTransmission</type>
             <joint name="${prefix}robotiq_85_left_knuckle_joint">
-                <hardwareInterface>hardware_interface/PositionJointInterface</hardwareInterface>
+                <hardwareInterface>hardware_interface/EffortJointInterface</hardwareInterface>
             </joint>
             <actuator name="${prefix}robotiq_85_left_knuckle_motor">
                 <mechanicalReduction>1</mechanicalReduction>
-                <hardwareInterface>hardware_interface/PositionJointInterface</hardwareInterface>
+                <hardwareInterface>hardware_interface/EffortJointInterface</hardwareInterface>
             </actuator>
         </transmission>
@@ -110,9 +110,11 @@
             <mu2>0.2</mu2>
             <selfCollide>false</selfCollide>
+            <!-- <dynamics damping="0.7" friction="100.0" /> -->
         </gazebo>
         <gazebo reference="${prefix}robotiq_85_left_finger_tip_link">
             <mu1>0.2</mu1>
             <mu2>0.2</mu2>
-            <selfCollide>true</selfCollide>
+            <selfCollide>false</selfCollide>
+            <!-- <dynamics damping="0.7" friction="100.0" /> -->
         </gazebo>
         <gazebo reference="${prefix}robotiq_85_left_knuckle_link">
@@ -120,4 +122,5 @@
             <mu2>0.2</mu2>
             <selfCollide>false</selfCollide>
+            <!-- <dynamics damping="0.7" friction="2.0" /> -->
         </gazebo>
         <gazebo reference="${prefix}robotiq_85_left_finger_link">
@@ -125,4 +128,5 @@
             <mu2>0.2</mu2>
             <selfCollide>false</selfCollide>
+            <!-- <dynamics damping="0.7" friction="100.0" /> -->
         </gazebo>
         <gazebo reference="${prefix}robotiq_85_right_inner_knuckle_link">
@@ -130,9 +134,11 @@
             <mu2>0.2</mu2>
             <selfCollide>false</selfCollide>
+            <!-- <dynamics damping="0.7" friction="100.0" /> -->
         </gazebo>
         <gazebo reference="${prefix}robotiq_85_right_finger_tip_link">
             <mu1>0.2</mu1>
             <mu2>0.2</mu2>
-            <selfCollide>true</selfCollide>
+            <selfCollide>false</selfCollide>
+            <!-- <dynamics damping="0.7" friction="100.0" /> -->
         </gazebo>
         <gazebo reference="${prefix}robotiq_85_right_knuckle_link">
@@ -140,4 +146,5 @@
             <mu2>0.2</mu2>
             <selfCollide>false</selfCollide>
+            <!-- <dynamics damping="0.7" friction="100.0" /> -->
         </gazebo>
         <gazebo reference="${prefix}robotiq_85_right_finger_link">
@@ -145,4 +152,5 @@
             <mu2>0.2</mu2>
             <selfCollide>false</selfCollide>
+            <!-- <dynamics damping="0.7" friction="100.0" /> -->
         </gazebo>
     </xacro:macro>

File: ws_capstone/src/urdf_descriptions_plugins/robotiq_85_description/urdf/robotiq_85_gripper.urdf.xacro (robot description, xacro)
@@ -35,4 +35,5 @@
             <origin rpy="${pi} 0.0 0.0" xyz="0.05490451627 0.03060114443 0.0"/>
             <limit lower="0.0" upper="0.8" velocity="2.0" effort="10"/>
+            <dynamics friction="9"/>
         </joint>
         <joint name="${prefix}robotiq_85_right_knuckle_joint" type="continuous">
@@ -41,6 +42,7 @@
             <axis xyz="0 0 1"/>
             <origin rpy="0.0 0.0 0.0" xyz="0.05490451627 -0.03060114443 0.0"/>
-            <limit lower="-3.14" upper="3.14" velocity="100.0" effort="1000"/>
+            <limit lower="-3.14" upper="3.14" velocity="2" effort="1000"/>
             <mimic joint="${prefix}robotiq_85_left_knuckle_joint"/>
+            <!-- <dynamics damping="0.7"/> -->
         </joint>
         <link name="${prefix}robotiq_85_left_knuckle_link">
@@ -89,4 +91,5 @@
             <!-- added -->
             <origin xyz="-0.00408552455 -0.03148604435 0.0" rpy="0 0 0" />
+            <!-- <dynamics damping="0.7"/> -->
         </joint>
         <joint name="${prefix}robotiq_85_right_finger_joint" type="continuous">
@@ -97,4 +100,5 @@
             <!-- added -->
             <origin xyz="-0.00408552455 -0.03148604435 0.0" rpy="0 0 0" />
+            <!-- <dynamics damping="0.7"/> -->
         </joint>
         <link name="${prefix}robotiq_85_left_finger_link">
@@ -141,6 +145,7 @@
             <axis xyz="0 0 1"/>
             <origin xyz="0.06142 0.0127 0" rpy="${pi} 0.0 0.0" />
-            <limit lower="-3.14" upper="3.14" velocity="100.0" effort="0.1"/>
+            <limit lower="-3.14" upper="3.14" velocity="2" effort="10"/>
             <mimic joint="${prefix}robotiq_85_left_knuckle_joint" offset="0"/>
+            <!-- <dynamics damping="0.7"/> -->
         </joint>
         <joint name="${prefix}robotiq_85_right_inner_knuckle_joint" type="continuous">
@@ -149,6 +154,7 @@
             <axis xyz="0 0 1"/>
             <origin xyz="0.06142 -0.0127 0" rpy="0 0 0"/>
-            <limit lower="-3.14" upper="3.14" velocity="100.0" effort="0.1"/>
+            <limit lower="-3.14" upper="3.14" velocity="2" effort="10"/>
             <mimic joint="${prefix}robotiq_85_left_knuckle_joint" offset="0"/>
+            <!-- <dynamics damping="0.7"/> -->
         </joint>
         <link name="${prefix}robotiq_85_left_inner_knuckle_link">
@@ -195,6 +201,7 @@
             <axis xyz="0 0 1"/>
             <origin xyz="0.04303959807 -0.03759940821 0.0" rpy="0.0 0.0 0.0"/>
-            <limit lower="-3.14" upper="3.14" velocity="100.0" effort="0.1"/>
+            <limit lower="-3.14" upper="3.14" velocity="2" effort="10"/>
             <mimic joint="${prefix}robotiq_85_left_knuckle_joint" multiplier="-1"/>
+            <!-- <dynamics damping="0.7"/> -->
         </joint>
         <joint name="${prefix}robotiq_85_right_finger_tip_joint" type="continuous">
@@ -203,6 +210,7 @@
             <axis xyz="0 0 1"/>
             <origin rpy="0.0 0.0 0.0" xyz="0.04303959807 -0.03759940821  0.0"/>
-            <limit lower="-3.14" upper="3.14" velocity="100.0" effort="0.1"/>
+            <limit lower="-3.14" upper="3.14" velocity="2" effort="10"/>
             <mimic joint="${prefix}robotiq_85_left_knuckle_joint" multiplier="-1"/>
+            <!-- <dynamics damping="0.7"/> -->
         </joint>
         <link name="${prefix}robotiq_85_left_finger_tip_link">

Commit message: upped gripper torque

File: ws_capstone/src/urdf_descriptions_plugins/robotiq_85_description/urdf/robotiq_85_gripper.transmission.xacro (robot description, xacro)
@@ -68,5 +68,5 @@
                 <joint>${prefix}robotiq_85_left_knuckle_joint</joint>
                 <mimicJoint>${prefix}robotiq_85_right_knuckle_joint</mimicJoint>
-                <maxEffort>9.01</maxEffort>
+                <maxEffort>20.01</maxEffort>
                 <!-- <multiplier>1.0</multiplier>
                 <offset>0.0</offset> -->
@@ -75,5 +75,5 @@
                 <joint>${prefix}robotiq_85_left_knuckle_joint</joint>
                 <mimicJoint>${prefix}robotiq_85_left_inner_knuckle_joint</mimicJoint>
-                <maxEffort>9.01</maxEffort>
+                <maxEffort>20.01</maxEffort>
                 <!-- <multiplier>1.0</multiplier>
                 <offset>0.0</offset> -->
@@ -82,5 +82,5 @@
                 <joint>${prefix}robotiq_85_left_knuckle_joint</joint>
                 <mimicJoint>${prefix}robotiq_85_right_inner_knuckle_joint</mimicJoint>
-                <maxEffort>9.01</maxEffort>
+                <maxEffort>20.01</maxEffort>
                 <!-- <multiplier>1.0</multiplier>
                 <offset>0.0</offset> -->
@@ -89,5 +89,5 @@
                 <joint>${prefix}robotiq_85_left_knuckle_joint</joint>
                 <mimicJoint>${prefix}robotiq_85_left_finger_tip_joint</mimicJoint>
-                <maxEffort>9.01</maxEffort>
+                <maxEffort>20.01</maxEffort>
                 <multiplier>-1.0</multiplier>
                 <!-- <offset>0.0</offset> -->
@@ -96,5 +96,5 @@
                 <joint>${prefix}robotiq_85_left_knuckle_joint</joint>
                 <mimicJoint>${prefix}robotiq_85_right_finger_tip_joint</mimicJoint>
-                <maxEffort>9.01</maxEffort>
+                <maxEffort>20.01</maxEffort>
                 <multiplier>-1.0</multiplier>
                 <!-- <offset>0.0</offset> -->

File: ws_capstone/src/urdf_descriptions_plugins/robotiq_85_description/urdf/robotiq_85_gripper.urdf.xacro (robot description, xacro)
@@ -34,5 +34,5 @@
             <axis xyz="0 0 1"/>
             <origin rpy="${pi} 0.0 0.0" xyz="0.05490451627 0.03060114443 0.0"/>
-            <limit lower="0.0" upper="0.8" velocity="2.0" effort="9.01"/>
+            <limit lower="0.0" upper="0.8" velocity="2.0" effort="20.01"/>
             <dynamics friction="9"/>
         </joint>
@@ -42,5 +42,5 @@
             <axis xyz="0 0 1"/>
             <origin rpy="0.0 0.0 0.0" xyz="0.05490451627 -0.03060114443 0.0"/>
-            <limit lower="-3.14" upper="3.14" velocity="2" effort="9.01"/>
+            <limit lower="-3.14" upper="3.14" velocity="2" effort="20.01"/>
             <mimic joint="${prefix}robotiq_85_left_knuckle_joint"/>
             <!-- <dynamics damping="0.7"/> -->
@@ -148,5 +148,5 @@
             <axis xyz="0 0 1"/>
             <origin xyz="0.06142 0.0127 0" rpy="${pi} 0.0 0.0" />
-            <limit lower="-3.14" upper="3.14" velocity="2" effort="9.01"/>
+            <limit lower="-3.14" upper="3.14" velocity="2" effort="20.01"/>
             <mimic joint="${prefix}robotiq_85_left_knuckle_joint" offset="0"/>
             <!-- <dynamics damping="0.7"/> -->
@@ -158,5 +158,5 @@
             <axis xyz="0 0 1"/>
             <origin xyz="0.06142 -0.0127 0" rpy="0 0 0"/>
-            <limit lower="-3.14" upper="3.14" velocity="2" effort="9.01"/>
+            <limit lower="-3.14" upper="3.14" velocity="2" effort="20.01"/>
             <mimic joint="${prefix}robotiq_85_left_knuckle_joint" offset="0"/>
             <!-- <dynamics damping="0.7"/> -->
@@ -206,5 +206,5 @@
             <axis xyz="0 0 1"/>
             <origin xyz="0.04303959807 -0.03759940821 0.0" rpy="0.0 0.0 0.0"/>
-            <limit lower="-3.14" upper="3.14" velocity="2" effort="9.01"/>
+            <limit lower="-3.14" upper="3.14" velocity="2" effort="20.01"/>
             <mimic joint="${prefix}robotiq_85_left_knuckle_joint" multiplier="-1"/>
             <!-- <dynamics damping="0.7"/> -->
@@ -216,5 +216,5 @@
             <axis xyz="0 0 1"/>
             <origin rpy="0.0 0.0 0.0" xyz="0.04303959807 -0.03759940821  0.0"/>
-            <limit lower="-3.14" upper="3.14" velocity="2" effort="9.01"/>
+            <limit lower="-3.14" upper="3.14" velocity="2" effort="20.01"/>
             <mimic joint="${prefix}robotiq_85_left_knuckle_joint" multiplier="-1"/>
             <!-- <dynamics damping="0.7"/> -->
